Commit message: Update code 13/3/26. complete FK, in-progress IK, and to do speed selection, joint limit, safety shutdown features

File: src/motor_node/urdf/arm.urdf (robot description, URDF)
Before this commit: robot robot_arm, 5 links, 4 joints
Joints:
- joint base_joint: axis 0 0 -1 -> 0 0 1
- joint elbow_joint: axis 1 0 0 -> -1 0 0; limit lower=-3.14 upper=3.14 -> lower=-6.28 upper=6.28; origin xyz=0.08 0 0.5 rpy=0 0 0 -> xyz=0.08 0 0.5 rpy=3.14 0 0
- joint shoulder_joint: limit lower=-1.57 upper=1.57 -> lower=0 upper=3.14; origin xyz=0 0 0.07 rpy=0 0 0 -> xyz=0 0 0.07 rpy=-1.57 0 0

Commit message: added end effector code

File: src/motor_node/urdf/arm.urdf (robot description, URDF)
Before this commit: robot robot_arm, 5 links, 4 joints
Joints:
- joint base_joint: axis 0 0 1 -> 0 0 -1

Commit message: joints limit, visualization, safety

File: src/motor_node/urdf/arm.urdf (robot description, URDF)
Before this commit: robot robot_arm, 5 links, 4 joints
Joints:
- joint base_joint: limit lower=-6.28 upper=6.28 -> lower=-3.14 upper=3.14
- joint elbow_joint: limit lower=-6.28 upper=6.28 -> lower=0 upper=4.71

Commit message: new urdf

File: src/motor_node/urdf/arm.urdf (robot description, URDF)
Before this commit: robot robot_arm, 8 links, 7 joints
Joints:
- joint ee_joint: origin xyz=0 0 0.05 rpy=0 0 0 -> xyz=0 0 -0.1 rpy=0 0 0
- joint pitch_joint: origin xyz=-0.05 -0.05 0 rpy=0 0 0 -> xyz=-0.05 0.05 0 rpy=0 0 0
- joint roll_joint: origin xyz=0 0 0.075 rpy=0 0 0 -> xyz=0 0 -0.075 rpy=0 0 0
- joint yaw_joint: axis 0 1 0 -> 0 -1 0; origin xyz=0 -0.05 0.6 rpy=0 0 0 -> xyz=0 0.05 0.6 rpy=0 0 0
